File: LoraTTNMapper/Eagle PCB/TBEAM_V10_Stack.brd (EAGLE design)
At the start: 100 x 80 mm, 13 parts, among them IC2 ULN2003AD, U1 GY-521MPU6050

Commit message: Gyro + PCB
Parts:
- moved U1 84.9 mm to (20.3, 59.7), turned to 270 degrees
- moved LED1 45.9 mm to (38.1, 63.5), turned to 180 degrees
- moved IC2 45.1 mm to (49.5, 63.5)
- moved R1 40.8 mm to (38.1, 66.0), turned to 0 degrees
- moved LED3 35.8 mm to (58.4, 53.3)
- moved LED2 35.7 mm to (48.3, 53.3)
- moved R2 28.0 mm to (52.1, 53.3), turned to 270 degrees
- moved R3 27.9 mm to (62.2, 53.3), turned to 270 degrees
- moved OLED_DISPLAY 21.6 mm to (52.1, 74.9)
- moved BME280 21.6 mm to (68.6, 74.9)
- moved SERVO_1 14.0 mm to (49.5, 45.7)
- moved JP2 14.0 mm to (59.7, 45.7)
- moved U$1 11.7 mm to (30.5, 63.5)
Connections:
- net N$1: now also U$1.23; no longer U$1.22
Routing:
- net GND: track 0.00 -> 140.7 mm
- net VDD: track 0.00 -> 72.4 mm
- net GPIO35: track 0.00 -> 55.4 mm
- net GPIO32: track 0.00 -> 51.5 mm
- net VDD_SWITCHABLE: track 0.00 -> 51.3 mm
- net SCL: track 0.00 -> 49.1 mm
- net SDA: track 0.00 -> 48.9 mm
- net GPIO15: track 0.00 -> 40.3 mm
- net N$2: track 0.00 -> 32.6 mm
- net N$6: track 0.00 -> 3.96 mm
- net N$5: track 0.00 -> 3.95 mm
- net N$4: track 0.00 -> 2.70 mm

Commit message: So long so good
Parts:
- removed JP2: Servo_2, pinhead:1X03
- added C1, C2: 100nF, rcl:C050-024X044
- added D1, D2, D3, D4, D5, D6, D7, D8: (no value), diode:D-5
- added IC1: L298, st-microelectronics:MULTIWATT-15
- added J1, J2, J3: 1X2-3.5MM, adafruit:1X2-3.5MM
- added SERVO_2: Servo_2, pinhead:1X03
- moved BME280 63.9 mm to (91.4, 15.2)
- moved OLED_DISPLAY 51.1 mm to (81.3, 33.0)
- moved LED2 47.9 mm to (73.7, 12.7)
- moved U1 46.8 mm to (50.8, 24.1)
- moved SERVO_1 44.9 mm to (71.1, 6.35)
- moved R2 44.4 mm to (69.8, 12.7)
- moved LED3 40.8 mm to (62.2, 12.7)
- moved R3 40.8 mm to (58.4, 12.7)
- moved R1 38.9 mm to (7.62, 41.9), turned to 90 degrees
- moved LED1 31.4 mm to (15.2, 41.9), turned to 90 degrees
- moved IC2 4.58 mm to (53.3, 61.0)
Connections:
- new net N$10: D5.A, D7.C, IC1.13, J3.1
- new net N$7: D1.A, D2.C, IC1.2, J2.1
- new net N$8: D3.A, D4.C, IC1.3, J2.2
- new net N$9: D6.A, D8.C, IC1.14, J3.2
- new net V+: C2.1, D1.C, D3.C, D5.C, D6.C, IC1.4, J1.1
- net +5V: now also C1.1, IC1.9
- net GND: now also C1.2, C2.2, D2.A, D4.A, D7.A, D8.A, IC1.1, IC1.15, IC1.8, J1.2
- net GPIO32: now also SERVO_2.3; no longer JP2.3
- net N$2: now also SERVO_2.1; no longer JP2.1
- net VDD: now also SERVO_2.2; no longer JP2.2
Routing:
- net GND: track 140.7 -> 0.00 mm
- net VDD: track 72.4 -> 0.00 mm
- net GPIO35: track 55.4 -> 0.00 mm
- net GPIO32: track 51.5 -> 0.00 mm
- net VDD_SWITCHABLE: track 51.3 -> 0.00 mm
- net SCL: track 49.1 -> 0.00 mm
- net SDA: track 48.9 -> 0.00 mm
- net GPIO15: track 40.3 -> 0.00 mm
- net N$2: track 32.6 -> 0.00 mm
- net N$6: track 3.96 -> 0.00 mm
- net N$5: track 3.95 -> 0.00 mm
- net N$4: track 2.70 -> 0.00 mm
Other:
- board text added: "+ 3-12Volt"
- board text added: "I2C Display"
- board text added: "Motor 1"
- board text added: "Motor 2"
- board text added: "Power Motor"
- board text added: "VDD Switchable"

Commit message: Board Layout
Parts:
- removed U1: GY-521MPU6050, gy-521:GY-521
- LED1: value (none) -> Power Rail
- moved OLED_DISPLAY 16.5 mm to (66.0, 39.4)
- moved R1 11.7 mm to (19.1, 39.4)
- moved LED1 9.67 mm to (19.1, 33.0)
- renumbered SERVO_2 to SERVO_2/GPIO32
Connections:
- removed net N$1: U$1.23, U1.INT
- net GND: no longer U1.GND
- net SCL: no longer U1.SCL
- net SDA: no longer U1.SDA
- net VDD: no longer U1.VCC
